Commit message: adjstments 11/12

File: bluerov2_description/urdf/bluerov2_alpha/bluerov2_alpha.xacro (robot description, xacro)
@@ -10,5 +10,5 @@
   <xacro:arg name="prefix" default="" />
   <xacro:arg name="use_sim" default="true" />
-  <xacro:arg name="description_package" default="bluerov2_cirtesu_core" />
+  <xacro:arg name="description_package" default="bluerov2_description" />
   <!-- Properties -->
   <xacro:property name="description_package" value="$(arg description_package)" />
@@ -18,6 +18,6 @@
   <xacro:include
     filename="$(find ${description_package})/urdf/bluerov2_alpha/urdf.xacro" />
-  <xacro:include
-    filename="$(find alpha_description)/xacro/alpha.ros2_control.xacro" />
+  <!-- <xacro:include
+    filename="$(find alpha_description)/xacro/alpha.ros2_control.xacro" /> -->
   <xacro:bluerov2_heavy_alpha_urdf
     prefix="${prefix}" />

File: bluerov2_description/urdf/bluerov2_alpha/urdf.xacro (robot description, xacro)
@@ -21,5 +21,5 @@
       </inertial>
     </link>
-    <link name="${prefix}ballast_link">
+    <!-- <link name="${prefix}ballast_link">
       <inertial>
         <mass value="0.0001" />
@@ -33,7 +33,4 @@
         />
       </inertial>
-      <!-- Split the collision into four boxes so that
-      we can adjust each one to balance things out -->
-      <!-- Front left -->
       <collision>
         <geometry>
@@ -42,5 +39,4 @@
         <origin rpy="0 0 0" xyz="0.11425 0.14375 0.08" />
       </collision>
-      <!-- Front right -->
       <collision>
         <geometry>
@@ -49,5 +45,4 @@
         <origin rpy="0 0 0" xyz="0.11425 -0.14375 0.08" />
       </collision>
-      <!-- Back right -->
       <collision>
         <geometry>
@@ -56,5 +51,5 @@
         <origin rpy="0 0 0" xyz="-0.11425 -0.14375 0.08" />
       </collision>
-    </link>
+    </link> -->
     <joint name="${prefix}manipulator_mount_joint" type="fixed">
       <origin rpy="0 0 -1.57" xyz="0.105 -0.21 0.07" />
@@ -62,12 +57,10 @@
       <child link="${prefix}manipulator_mount_link" />
     </joint>
-    <joint name="${prefix}ballast_joint" type="fixed">
+    <!-- <joint name="${prefix}ballast_joint" type="fixed">
       <origin rpy="0 0 0" xyz="0 0 0" />
       <parent link="${prefix}base_link" />
       <child link="${prefix}ballast_link" />
-    </joint>
+    </joint> -->
     <!-- Imports -->
-    <!-- <xacro:include filename="$(find alpha_description)/xacro/alpha.urdf.xacro" /> -->
-    <xacro:include filename="$(find bluerov2_cirtesu_core)/urdf/bluerov2_heavy/urdf_payload.xacro" />
     <!-- Instantiate the Alpha -->
     <!-- <xacro:alpha_urdf

File: bluerov2_description/urdf/bluerov2_heavy/bluerov2.xacro (robot description, xacro)
@@ -1,7 +1,7 @@
 <?xml version="1.0"?>
 <robot name="bluerov2_heavy" xmlns:xacro="http://ros.org/wiki/xacro">
-  <xacro:arg name="prefix" default="bluerov/" />
+  <xacro:arg name="prefix" default="" />
   <!-- Import BlueROV2 macro -->
-  <xacro:include filename="$(find bluerov2_cirtesu_core)/urdf/bluerov2_heavy/urdf_payload.xacro" />
+  <xacro:include filename="$(find bluerov2_description)/urdf/bluerov2_heavy/urdf_payload.xacro" />
   <xacro:bluerov2_heavy_urdf prefix="$(arg prefix)" />
 </robot>

File: bluerov2_description/urdf/bluerov2_heavy/urdf.xacro (robot description, xacro)
@@ -18,5 +18,5 @@
         <geometry>
           <mesh
-            filename="file://$(find bluerov2_cirtesu_core)/resources/bluerov2_heavy/bluerov2_heavy.dae"
+            filename="file://$(find bluerov2_description)/resources/bluerov2_heavy/bluerov2_heavy.dae"
             scale="0.025 0.025 0.025"
           />
@@ -45,5 +45,5 @@
     </xacro:camera_urdf-->
     <!-- Import T200 macro -->
-    <xacro:include filename="$(find bluerov2_cirtesu_core)/urdf/t200/urdf.xacro" />
+    <xacro:include filename="$(find bluerov2_description)/urdf/t200/urdf.xacro" />
     <xacro:t200_urdf parent="${prefix}base_link" prefix="${prefix}" ccw="true" id="1">
       <origin rpy="-1.571 1.571 -0.785" xyz="0.14 -0.092 0.0" />

File: bluerov2_description/urdf/bluerov2_heavy/urdf_payload.xacro (robot description, xacro)
@@ -18,5 +18,5 @@
         <geometry>
           <mesh
-            filename="file://$(find bluerov2_cirtesu_core)/resources/bluerov2_heavy/bluerov2_heavy.dae"
+            filename="file://$(find bluerov2_description)/resources/bluerov2_heavy/bluerov2_heavy.dae"
             scale="0.025 0.025 0.025"
           />
@@ -69,5 +69,5 @@
     </xacro:camera_urdf-->
     <!-- Import T200 macro -->
-    <xacro:include filename="$(find bluerov2_cirtesu_core)/urdf/t200/urdf.xacro" />
+    <xacro:include filename="$(find bluerov2_description)/urdf/t200/urdf.xacro" />
     <xacro:t200_urdf parent="${prefix}base_link" prefix="${prefix}" ccw="true" id="1">
       <origin rpy="-1.571 1.571 -0.785" xyz="0.14 -0.092 0.0" />

File: bluerov2_description/urdf/t200/urdf.xacro (robot description, xacro)
@@ -17,10 +17,10 @@
         <xacro:if value="${ccw}">
           <geometry>
-            <mesh filename="file://$(find bluerov2_cirtesu_core)/resources/t200/ccw_prop.dae" />
+            <mesh filename="file://$(find bluerov2_description)/resources/t200/ccw_prop.dae" />
           </geometry>
         </xacro:if>
         <xacro:unless value="${ccw}">
           <geometry>
-            <mesh filename="file://$(find bluerov2_cirtesu_core)/resources/t200/cw_prop.dae" />
+            <mesh filename="file://$(find bluerov2_description)/resources/t200/cw_prop.dae" />
           </geometry>
         </xacro:unless>
